Commit message: feat: sync DR02 finetuned assets

File: source/robot_lab/data/Robots/deeprobotics/dr02_pro_description/urdf/dr02_pro.urdf (robot description, URDF)
Before this commit: robot DR02-pro, 40 links, 39 joints
Joints:
- joint neck_y_joint: axis 0 1 0 -> (none); limit lower=-0.349066 upper=0.349066 effort=50 velocity=23.76 -> (none); type revolute -> fixed
- joint neck_z_joint: axis 0 0 1 -> (none); limit lower=-1.745329 upper=3.665191 effort=50 velocity=23.76 -> (none); type revolute -> fixed
